File: motor-controller-pcb/motor-controller-pcb.kicad_sch (KiCad schematic)
At the start: 25 parts, among them J1 Motor 1, J10 3V3, J11 Conn_01x05_Pin, J2 Motor 2, J3 Motor 3, J4 Motor 4, J5 Dribbler Motor, J6 Battery Connector, J7 GND, J8 5V, J9 V_Batt, SW1 Battery Switch

Commit message: feat: pcb layout
Parts:
- J1, J2, J3, J4, J5: symbol Connector_Generic_MountingPin:Conn_01x06_MountingPin -> Connector:Conn_01x06_Pin
- J6, SW1: footprint Connector_Wire:SolderWire-6sqmm_1x02_P14mm_D3.5mm_OD7mm_Relief2x -> Connector_Wire:SolderWire-2sqmm_1x02_P7.8mm_D2mm_OD3.9mm_Relief2x
- U1, U2, U3: footprint (none) -> robocup-library:DRI044
Connections:
- no-connect marks 21 -> 16
Changed lines of the file:
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@@
 	)
 	(no_connect
-		(at 27.94 90.17)
-	)
-	(no_connect
 		(at 55.88 151.13)
 	)
@@
 	)
 	(no_connect
-		(at 27.94 49.53)
-	)
-	(no_connect
 		(at 55.88 146.05)
 	)
@@
 	)
 	(no_connect
-		(at 50.8 158.75)
-	)
-	(no_connect
 		(at 214.63 114.3)
 	)
@@
 		(at 214.63 104.14)
 	)
-	(no_connect
-		(at 27.94 69.85)
-	)
-	(no_connect
-		(at 27.94 110.49)
-	)
 	(wire
 		(pts
@@
 	)
 	(symbol
-		(lib_id "Connector_Generic_MountingPin:Conn_01x06_MountingPin")
+		(lib_id "Connector:Conn_01x06_Pin")
 		(at 27.94 97.79 0)
-		(mirror y)
 		(unit 1)
 		(exclude_from_sim no)
@@
 		(dnp no)
 		(property "Reference" "J4"
-			(at 25.4 98.1455 0)
+			(at 22.098 96.012 0)
 			(effects
 				(font
@@
 		)
 		(property "Value" "Motor 4"
-			(at 25.4 100.6855 0)
+			(at 19.304 98.298 0)
 			(effects
 				(font
@@
 			)
 		)
-		(property "Description" "Generic connectable mounting pin connector, single row, 01x06, script generated (kicad-library-utils/schlib/autogen/connector/)"
+		(property "Description" "Generic connector, single row, 01x06, script generated"
 			(at 27.94 97.79 0)
 			(effects
@@
 		(pin "4"
 		)
-		(pin "MP"
-		)
 		(instances
 			(project ""
@@
 	)
 	(symbol
-		(lib_id "Connector_Generic_MountingPin:Conn_01x06_MountingPin")
+		(lib_id "Connector:Conn_01x06_Pin")
 		(at 50.8 146.05 0)
-		(mirror y)
 		(unit 1)
 		(exclude_from_sim no)
@@
 		(on_board yes)
 		(dnp no)
-		(fields_autoplaced yes)
 		(property "Reference" "J5"
-			(at 50.8 134.62 0)
+			(at 42.164 146.812 0)
 			(effects
 				(font
 					(size 1.27 1.27)
 				)
+				(justify right)
 			)
 		)
 		(property "Value" "Dribbler Motor"
-			(at 50.8 137.16 0)
+			(at 48.006 148.844 0)
 			(effects
 				(font
 					(size 1.27 1.27)
 				)
+				(justify right)
 			)
 		)
@@
 			)
 		)
-		(property "Description" "Generic connectable mounting pin connector, single row, 01x06, script generated (kicad-library-utils/schlib/autogen/connector/)"
+		(property "Description" "Generic connector, single row, 01x06, script generated"
 			(at 50.8 146.05 0)
 			(effects
@@
 		(pin "6"
 		)
-		(pin "MP"
-		)
 		(pin "5"
 		)
@@
 	)
 	(symbol
-		(lib_id "Connector_Generic_MountingPin:Conn_01x06_MountingPin")
+		(lib_id "Connector:Conn_01x06_Pin")
 		(at 27.94 57.15 0)
-		(mirror y)
 		(unit 1)
 		(exclude_from_sim no)
@@
 		(dnp no)
 		(property "Reference" "J2"
-			(at 25.4 57.5055 0)
+			(at 21.59 56.896 0)
 			(effects
 				(font
@@
 		)
 		(property "Value" "Motor 2"
-			(at 25.4 60.0455 0)
+			(at 18.542 58.928 0)
 			(effects
 				(font
@@
 			)
 		)
-		(property "Description" "Generic connectable mounting pin connector, single row, 01x06, script generated (kicad-library-utils/schlib/autogen/connector/)"
+		(property "Description" "Generic connector, single row, 01x06, script generated"
 			(at 27.94 57.15 0)
 			(effects
@@
 		(pin "4"
 		)
-		(pin "MP"
-		)
 		(instances
 			(project ""
@@
 	)
 	(symbol
-		(lib_id "Connector_Generic_MountingPin:Conn_01x06_MountingPin")
+		(lib_id "Connector:Conn_01x06_Pin")
 		(at 27.94 36.83 0)
-		(mirror y)
 		(unit 1)
 		(exclude_from_sim no)
@@
 		(dnp no)
 		(property "Reference" "J1"
-			(at 25.4 37.1855 0)
+			(at 21.59 37.592 0)
 			(effects
 				(font
@@
 		)
 		(property "Value" "Motor 1"
-			(at 25.4 39.7255 0)
+			(at 19.05 40.132 0)
 			(effects
 				(font
@@
 			)
 		)
-		(property "Description" "Generic connectable mounting pin connector, single row, 01x06, script generated (kicad-library-utils/schlib/autogen/connector/)"
+		(property "Description" "Generic connector, single row, 01x06, script generated"
 			(at 27.94 36.83 0)
 			(effects
@@
 		(pin "4"
 		)
-		(pin "MP"
-		)
 		(instances
 			(project ""
@@
 			)
 		)
-		(property "Footprint" ""
+		(property "Footprint" "robocup-library:DRI044"
 			(at 91.44 38.1 0)
 			(effects
@@
 	)
 	(symbol
-		(lib_id "Connector_Generic_MountingPin:Conn_01x06_MountingPin")
+		(lib_id "Connector:Conn_01x06_Pin")
 		(at 27.94 77.47 0)
-		(mirror y)
 		(unit 1)
 		(exclude_from_sim no)
@@
 		(dnp no)
 		(property "Reference" "J3"
-			(at 25.4 77.8255 0)
+			(at 22.098 77.978 0)
 			(effects
 				(font
@@
 		)
 		(property "Value" "Motor 3"
-			(at 25.4 80.3655 0)
+			(at 18.796 80.01 0)
 			(effects
 				(font
@@
 			)
 		)
-		(property "Description" "Generic connectable mounting pin connector, single row, 01x06, script generated (kicad-library-utils/schlib/autogen/connector/)"
+		(property "Description" "Generic connector, single row, 01x06, script generated"
 			(at 27.94 77.47 0)
 			(effects
@@
 		(pin "4"
 		)
-		(pin "MP"
-		)
 		(instances
 			(project ""
@@
 			)
 		)
-		(property "Footprint" ""
+		(property "Footprint" "robocup-library:DRI044"
 			(at 76.2 147.32 0)
 			(effects
@@
 			)
 		)
-		(property "Footprint" "Connector_Wire:SolderWire-6sqmm_1x02_P14mm_D3.5mm_OD7mm_Relief2x"
+		(property "Footprint" "Connector_Wire:SolderWire-2sqmm_1x02_P7.8mm_D2mm_OD3.9mm_Relief2x"
 			(at 25.4 199.39 0)
 			(effects
@@
 			)
 		)
-		(property "Footprint" "Connector_Wire:SolderWire-6sqmm_1x02_P14mm_D3.5mm_OD7mm_Relief2x"
+		(property "Footprint" "Connector_Wire:SolderWire-2sqmm_1x02_P7.8mm_D2mm_OD3.9mm_Relief2x"
 			(at 53.34 199.39 0)
 			(effects
@@
 			)
 		)
-		(property "Footprint" ""
+		(property "Footprint" "robocup-library:DRI044"
 			(at 92.71 78.74 0)
 			(effects

Commit message: feat: final
Parts:
- added J12: V_Batt, TerminalBlock:TerminalBlock_MaiXu_MX126-5.0-02P_1x02_P5.00mm, symbol Connector:Conn_01x02_Pin
Connections:
- net +BATT: now also J12.1 (Pin_1)
- net GND: now also J12.2 (Pin_2)
Changed lines of the file:
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@@
 	)
 	(junction
+		(at 171.45 218.44)
+		(diameter 0)
+		(color 0 0 0 0)
+	)
+	(junction
 		(at 186.69 208.28)
 		(diameter 0)
@@
 	(wire
 		(pts
+			(xy 171.45 218.44) (xy 171.45 224.79)
+		)
+		(stroke
+			(width 0)
+			(type default)
+		)
+	)
+	(wire
+		(pts
 			(xy 118.11 48.26) (xy 91.44 48.26)
 		)
@@
 	)
 	(symbol
+		(lib_id "power:GND")
+		(at 171.45 227.33 0)
+		(unit 1)
+		(exclude_from_sim no)
+		(in_bom yes)
+		(on_board yes)
+		(dnp no)
+		(fields_autoplaced yes)
+		(property "Reference" "#PWR030"
+			(at 171.45 233.68 0)
+			(effects
+				(font
+					(size 1.27 1.27)
+				)
+				(hide yes)
+			)
+		)
+		(property "Value" "GND"
+			(at 171.45 232.41 0)
+			(effects
+				(font
+					(size 1.27 1.27)
+				)
+			)
+		)
+		(property "Footprint" ""
+			(at 171.45 227.33 0)
+			(effects
+				(font
+					(size 1.27 1.27)
+				)
+				(hide yes)
+			)
+		)
+		(property "Datasheet" ""
+			(at 171.45 227.33 0)
+			(effects
+				(font
+					(size 1.27 1.27)
+				)
+				(hide yes)
+			)
+		)
+		(property "Description" "Power symbol creates a global label with name \"GND\" , ground"
+			(at 171.45 227.33 0)
+			(effects
+				(font
+					(size 1.27 1.27)
+				)
+				(hide yes)
+			)
+		)
+		(pin "1"
+		)
+		(instances
+			(project "motor-controller-pcb"
+				(path "/521a5f8e-be65-4be3-9b63-a6be4ecbc76a"
+					(reference "#PWR030")
+					(unit 1)
+				)
+			)
+		)
+	)
+	(symbol
 		(lib_id "Connector:Conn_01x06_Pin")
 		(at 27.94 97.79 0)
@@
 					(unit 1)
 				)
+			)
+		)
+	)
+	(symbol
+		(lib_id "Connector:Conn_01x02_Pin")
+		(at 166.37 224.79 0)
+		(unit 1)
+		(exclude_from_sim no)
+		(in_bom yes)
+		(on_board yes)
+		(dnp no)
+		(property "Reference" "J12"
+			(at 161.798 224.536 0)
+			(effects
+				(font
+					(size 1.27 1.27)
+				)
+			)
+		)
+		(property "Value" "V_Batt"
+			(at 161.544 226.822 0)
+			(effects
+				(font
+					(size 1.27 1.27)
+				)
+			)
+		)
+		(property "Footprint" "TerminalBlock:TerminalBlock_MaiXu_MX126-5.0-02P_1x02_P5.00mm"
+			(at 166.37 224.79 0)
+			(effects
+				(font
+					(size 1.27 1.27)
+				)
+				(hide yes)
+			)
+		)
+		(property "Datasheet" "~"
+			(at 166.37 224.79 0)
+			(effects
+				(font
+					(size 1.27 1.27)
+				)
+				(hide yes)
+			)
+		)
+		(property "Description" "Generic connector, single row, 01x02, script generated"
+			(at 166.37 224.79 0)
+			(effects
+				(font
+					(size 1.27 1.27)
+				)
+				(hide yes)
+			)
+		)
+		(pin "1"
+		)
+		(pin "2"
+		)
+		(instances
+			(project ""
+				(path "/521a5f8e-be65-4be3-9b63-a6be4ecbc76a"
+					(reference "J12")
+					(unit 1)
+				)

Commit message: feat: pcb prettification
Parts:
- U1, U2, U3: footprint robocup-library:DRI044 -> robocup-library:DRI0044
Changed lines of the file:
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@@
 			)
 		)
-		(property "Footprint" "robocup-library:DRI044"
+		(property "Footprint" "robocup-library:DRI0044"
 			(at 91.44 38.1 0)
 			(effects
@@
 			)
 		)
-		(property "Footprint" "robocup-library:DRI044"
+		(property "Footprint" "robocup-library:DRI0044"
 			(at 76.2 147.32 0)
 			(effects
@@
 			)
 		)
-		(property "Footprint" "robocup-library:DRI044"
+		(property "Footprint" "robocup-library:DRI0044"
 			(at 92.71 78.74 0)
 			(effects

Commit message: fix: make wire strain relief holes large enough
Parts:
- J6, SW1: footprint Connector_Wire:SolderWire-2sqmm_1x02_P7.8mm_D2mm_OD3.9mm_Relief2x -> Connector_Wire:SolderWire-4sqmm_1x02_P12mm_D3mm_OD6mm_Relief
Changed lines of the file:
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@@
 			)
 		)
-		(property "Footprint" "Connector_Wire:SolderWire-2sqmm_1x02_P7.8mm_D2mm_OD3.9mm_Relief2x"
+		(property "Footprint" "Connector_Wire:SolderWire-4sqmm_1x02_P12mm_D3mm_OD6mm_Relief"
 			(at 25.4 199.39 0)
 			(effects
@@
 			)
 		)
-		(property "Footprint" "Connector_Wire:SolderWire-2sqmm_1x02_P7.8mm_D2mm_OD3.9mm_Relief2x"
+		(property "Footprint" "Connector_Wire:SolderWire-4sqmm_1x02_P12mm_D3mm_OD6mm_Relief"
 			(at 53.34 199.39 0)
 			(effects
